File: electronics/scorbot_jcb/scorbot_jcb.brd (EAGLE design)
At the start: 100 x 80 mm, 5 parts

Commit message: Current sensor
Parts:
- added C1: (no value), rcl:C025-025X050
- HBRIDGE, XMC4800: value ARDUINO_R3_SHIELD -> ARDUINO_R3_SHIELDONLY_PADS; device uchile_robotics_eagle_lib:UNO_R3_SHIELD -> uchile_robotics_eagle_lib:UNO_R3_SHIELD_ONLY_PADS
- moved HB_OUT 192.2 mm to (94.0, 33.0)
- moved DB9 182.9 mm to (63.5, 10.2)
- moved CURRENT_SENSOR 139.9 mm to (43.2, 12.7)
- moved XMC4800 21.6 mm to (86.4, 25.4)
Connections:
- removed net VDD: CURRENT_SENSOR.2
- new net +3V3: C1.1, CURRENT_SENSOR.2, XMC4800.3.3V
- net +5V: now also XMC4800.5V
- net GND: now also C1.2, XMC4800.GND@0, XMC4800.GND@1, XMC4800.GND@2
Changed lines of the file:
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@@
 </autorouter>
 <elements>
-<element name="CURRENT_SENSOR" library="uchile_robotics_eagle_lib" package="TLI4970_D025T5" value="TLI4970_D025T5" x="-74.93" y="87.63"/>
-<element name="DB9" library="uchile_robotics_eagle_lib" package="XM3-LS" value="SCORBOT_CONNECTOR" x="-43.18" y="158.75"/>
-<element name="HBRIDGE" library="uchile_robotics_eagle_lib" package="UNO_R3_SHIELD" value="ARDUINO_R3_SHIELD" x="8.89" y="11.43"/>
-<element name="HB_OUT" library="uchile_robotics_eagle_lib" package="METALTEX-2S" value="METALTEX-2SHORT" x="-54.61" y="154.94"/>
-<element name="XMC4800" library="uchile_robotics_eagle_lib" package="UNO_R3_SHIELD" value="ARDUINO_R3_SHIELD" x="107.95" y="24.13" rot="R90"/>
+<element name="CURRENT_SENSOR" library="uchile_robotics_eagle_lib" package="TLI4970_D025T5" value="TLI4970_D025T5" x="43.18" y="12.7"/>
+<element name="DB9" library="uchile_robotics_eagle_lib" package="XM3-LS" value="SCORBOT_CONNECTOR" x="63.5" y="10.16"/>
+<element name="HBRIDGE" library="uchile_robotics_eagle_lib" package="UNO_R3_SHIELD_ONLY_PADS" value="ARDUINO_R3_SHIELDONLY_PADS" x="8.89" y="11.43"/>
+<element name="HB_OUT" library="uchile_robotics_eagle_lib" package="METALTEX-2S" value="METALTEX-2SHORT" x="93.98" y="33.02"/>
+<element name="XMC4800" library="uchile_robotics_eagle_lib" package="UNO_R3_SHIELD_ONLY_PADS" value="ARDUINO_R3_SHIELDONLY_PADS" x="86.36" y="25.4" rot="R90"/>
+<element name="C1" library="rcl" package="C025-025X050" value="" x="3.81" y="-3.81"/>
 </elements>
 <signals>
 <signal name="+5V">
 <contactref element="DB9" pad="P3"/>
+<contactref element="XMC4800" pad="5V"/>
+<wire x1="76" y1="11.1125" x2="57.15" y2="76.2" width="0" layer="19" extent="1-1"/>
 </signal>
 <signal name="GND">
 <contactref element="DB9" pad="P5"/>
 <contactref element="CURRENT_SENSOR" pad="1"/>
-<wire x1="-77.43" y1="84.13" x2="-36.16" y2="159.7025" width="0" layer="19" extent="1-1"/>
-</signal>
-<signal name="VDD">
-<contactref element="CURRENT_SENSOR" pad="2"/>
+<contactref element="XMC4800" pad="GND@0"/>
+<contactref element="XMC4800" pad="GND@1"/>
+<contactref element="XMC4800" pad="GND@2"/>
+<contactref element="C1" pad="2"/>
+<wire x1="52.07" y1="76.2" x2="54.61" y2="76.2" width="0" layer="19" extent="1-1"/>
+<wire x1="68.58" y1="27.94" x2="54.61" y2="76.2" width="0" layer="19" extent="1-1"/>
+<wire x1="70.52" y1="11.1125" x2="68.58" y2="27.94" width="0" layer="19" extent="1-1"/>
+<wire x1="40.68" y1="9.2" x2="70.52" y2="11.1125" width="0" layer="19" extent="1-1"/>
+<wire x1="5.08" y1="-3.81" x2="40.68" y2="9.2" width="0" layer="19" extent="1-1"/>
 </signal>
 <signal name="N$1">
 <contactref element="CURRENT_SENSOR" pad="8"/>
 <contactref element="DB9" pad="P9"/>
-<wire x1="-76.71" y1="90.1" x2="-34.49" y2="157.7975" width="0" layer="19" extent="1-1"/>
+<wire x1="41.4" y1="15.17" x2="72.19" y2="9.2075" width="0" layer="19" extent="1-1"/>
 </signal>
 <signal name="N$2">
@@
 <contactref element="HB_OUT" pad="P2"/>
 <contactref element="DB9" pad="P1"/>
-<wire x1="-52.07" y1="156.718" x2="-25.2" y2="159.7025" width="0" layer="19" extent="1-1"/>
+<wire x1="96.52" y1="34.798" x2="81.48" y2="11.1125" width="0" layer="19" extent="1-1"/>
+</signal>
+<signal name="+3V3">
+<contactref element="XMC4800" pad="3.3V"/>
+<contactref element="CURRENT_SENSOR" pad="2"/>
+<contactref element="C1" pad="1"/>
+<wire x1="41.98" y1="9.2" x2="59.69" y2="76.2" width="0" layer="19" extent="1-1"/>
+<wire x1="2.54" y1="-3.81" x2="41.98" y2="9.2" width="0" layer="19" extent="1-1"/>
 </signal>
 </signals>

Commit message: Schematic for shield
Parts:
- added R1, R2, R3: 1k, rcl:0309/12
- added R4, R5, R6: 2k, rcl:0309/12
Connections:
- new net !CS: CURRENT_SENSOR.5, XMC4800.D10
- new net ENC_A: R2.1, R5.2, XMC4800.D2
- new net ENC_B: R3.1, R6.2, XMC4800.D3
- new net HOME: R1.1, R4.2, XMC4800.D8
- new net IN1: HBRIDGE.D3, XMC4800.D6
- new net IN2: HBRIDGE.D11, XMC4800.D5
- new net INH1: HBRIDGE.D12, XMC4800.D4
- new net INH2: HBRIDGE.D13, XMC4800.D7
- new net MISO: CURRENT_SENSOR.3, XMC4800.D12
- new net N$10: DB9.P6, R2.2
- new net N$11: DB9.P8, R3.2
- new net N$9: DB9.P4, R1.2
- new net SCLK: CURRENT_SENSOR.4, XMC4800.D13
- net GND: now also HBRIDGE.GND@0, HBRIDGE.GND@1, R4.1, R5.1, R6.1
- net N$2: now also HB_OUT.P1
Changed lines of the file:
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@@
 <?xml version="1.0" encoding="utf-8"?>
 <!DOCTYPE eagle SYSTEM "eagle.dtd">
-<eagle version="7.4.0">
+<eagle version="7.6.0">
 <drawing>
 <settings>
@@
 <layers>
 <layer number="1" name="Top" color="4" fill="1" visible="yes" active="yes"/>
+<layer number="2" name="Route2" color="1" fill="3" visible="no" active="no"/>
+<layer number="3" name="Route3" color="4" fill="3" visible="no" active="no"/>
+<layer number="4" name="Route4" color="1" fill="4" visible="no" active="no"/>
+<layer number="5" name="Route5" color="4" fill="4" visible="no" active="no"/>
+<layer number="6" name="Route6" color="1" fill="8" visible="no" active="no"/>
+<layer number="7" name="Route7" color="4" fill="8" visible="no" active="no"/>
+<layer number="8" name="Route8" color="1" fill="2" visible="no" active="no"/>
+<layer number="9" name="Route9" color="4" fill="2" visible="no" active="no"/>
+<layer number="10" name="Route10" color="1" fill="7" visible="no" active="no"/>
+<layer number="11" name="Route11" color="4" fill="7" visible="no" active="no"/>
+<layer number="12" name="Route12" color="1" fill="5" visible="no" active="no"/>
+<layer number="13" name="Route13" color="4" fill="5" visible="no" active="no"/>
+<layer number="14" name="Route14" color="1" fill="6" visible="no" active="no"/>
+<layer number="15" name="Route15" color="4" fill="6" visible="no" active="no"/>
 <layer number="16" name="Bottom" color="1" fill="1" visible="yes" active="yes"/>
 <layer number="17" name="Pads" color="2" fill="1" visible="yes" active="yes"/>
@@
 <element name="XMC4800" library="uchile_robotics_eagle_lib" package="UNO_R3_SHIELD_ONLY_PADS" value="ARDUINO_R3_SHIELDONLY_PADS" x="86.36" y="25.4" rot="R90"/>
 <element name="C1" library="rcl" package="C025-025X050" value="" x="3.81" y="-3.81"/>
+<element name="R1" library="rcl" package="0309/12" value="1k" x="7.62" y="-8.89"/>
+<element name="R2" library="rcl" package="0309/12" value="1k" x="7.62" y="-15.24"/>
+<element name="R3" library="rcl" package="0309/12" value="1k" x="7.62" y="-21.59"/>
+<element name="R4" library="rcl" package="0309/12" value="2k" x="7.62" y="-27.94"/>
+<element name="R5" library="rcl" package="0309/12" value="2k" x="7.62" y="-34.29"/>
+<element name="R6" library="rcl" package="0309/12" value="2k" x="7.62" y="-40.64"/>
 </elements>
 <signals>
@@
 <contactref element="XMC4800" pad="GND@2"/>
 <contactref element="C1" pad="2"/>
+<contactref element="R4" pad="1"/>
+<contactref element="R5" pad="1"/>
+<contactref element="R6" pad="1"/>
+<contactref element="HBRIDGE" pad="GND@1"/>
+<contactref element="HBRIDGE" pad="GND@0"/>
 <wire x1="52.07" y1="76.2" x2="54.61" y2="76.2" width="0" layer="19" extent="1-1"/>
-<wire x1="68.58" y1="27.94" x2="54.61" y2="76.2" width="0" layer="19" extent="1-1"/>
+<wire x1="59.69" y1="45.72" x2="54.61" y2="76.2" width="0" layer="19" extent="1-1"/>
+<wire x1="59.69" y1="43.18" x2="59.69" y2="45.72" width="0" layer="19" extent="1-1"/>
+<wire x1="68.58" y1="27.94" x2="59.69" y2="43.18" width="0" layer="19" extent="1-1"/>
 <wire x1="70.52" y1="11.1125" x2="68.58" y2="27.94" width="0" layer="19" extent="1-1"/>
 <wire x1="40.68" y1="9.2" x2="70.52" y2="11.1125" width="0" layer="19" extent="1-1"/>
 <wire x1="5.08" y1="-3.81" x2="40.68" y2="9.2" width="0" layer="19" extent="1-1"/>
+<wire x1="1.27" y1="-27.94" x2="5.08" y2="-3.81" width="0" layer="19" extent="1-1"/>
+<wire x1="1.27" y1="-34.29" x2="1.27" y2="-27.94" width="0" layer="19" extent="1-1"/>
+<wire x1="1.27" y1="-40.64" x2="1.27" y2="-34.29" width="0" layer="19" extent="1-1"/>
 </signal>
 <signal name="N$1">
@@
 <signal name="N$2">
 <contactref element="CURRENT_SENSOR" pad="7"/>
+<contactref element="HB_OUT" pad="P1"/>
+<wire x1="44.96" y1="15.17" x2="91.44" y2="34.798" width="0" layer="19" extent="1-1"/>
 </signal>
 <signal name="N$3">
@@
 <wire x1="2.54" y1="-3.81" x2="41.98" y2="9.2" width="0" layer="19" extent="1-1"/>
 </signal>
+<signal name="MISO">
+<contactref element="XMC4800" pad="D12"/>
+<contactref element="CURRENT_SENSOR" pad="3"/>
+<wire x1="42.78" y1="9.2" x2="63.5" y2="27.94" width="0" layer="19" extent="1-1"/>
+</signal>
+<signal name="!CS">
+<contactref element="XMC4800" pad="D10"/>
+<contactref element="CURRENT_SENSOR" pad="5"/>
+<wire x1="44.38" y1="9.2" x2="58.42" y2="27.94" width="0" layer="19" extent="1-1"/>
+</signal>
+<signal name="SCLK">
+<contactref element="CURRENT_SENSOR" pad="4"/>
+<contactref element="XMC4800" pad="D13"/>
+<wire x1="43.58" y1="9.2" x2="66.04" y2="27.94" width="0" layer="19" extent="1-1"/>
+</signal>
+<signal name="IN1">
+<contactref element="XMC4800" pad="D6"/>
+<contactref element="HBRIDGE" pad="D3"/>
+<wire x1="11.43" y1="58.42" x2="46.99" y2="27.94" width="0" layer="19" extent="1-1"/>
+</signal>
+<signal name="IN2">
+<contactref element="XMC4800" pad="D5"/>
+<contactref element="HBRIDGE" pad="D11"/>
+<wire x1="11.43" y1="36.83" x2="44.45" y2="27.94" width="0" layer="19" extent="1-1"/>
+</signal>
+<signal name="INH1">
+<contactref element="XMC4800" pad="D4"/>
+<contactref element="HBRIDGE" pad="D12"/>
+<wire x1="11.43" y1="34.29" x2="41.91" y2="27.94" width="0" layer="19" extent="1-1"/>
+</signal>
+<signal name="INH2">
+<contactref element="XMC4800" pad="D7"/>
+<contactref element="HBRIDGE" pad="D13"/>
+<wire x1="11.43" y1="31.75" x2="49.53" y2="27.94" width="0" layer="19" extent="1-1"/>
+</signal>
+<signal name="N$9">
+<contactref element="DB9" pad="P4"/>
+<contactref element="R1" pad="2"/>
+<wire x1="13.97" y1="-8.89" x2="73.26" y2="11.1125" width="0" layer="19" extent="1-1"/>
+</signal>
+<signal name="N$10">
+<contactref element="R2" pad="2"/>
+<contactref element="DB9" pad="P6"/>
+<wire x1="13.97" y1="-15.24" x2="79.81" y2="9.2075" width="0" layer="19" extent="1-1"/>
+</signal>
+<signal name="N$11">
+<contactref element="DB9" pad="P8"/>
+<contactref element="R3" pad="2"/>
+<wire x1="13.97" y1="-21.59" x2="74.73" y2="9.2075" width="0" layer="19" extent="1-1"/>
+</signal>
+<signal name="HOME">
+<contactref element="XMC4800" pad="D8"/>
+<contactref element="R4" pad="2"/>
+<contactref element="R1" pad="1"/>
+<wire x1="1.27" y1="-8.89" x2="53.34" y2="27.94" width="0" layer="19" extent="1-1"/>
+<wire x1="13.97" y1="-27.94" x2="1.27" y2="-8.89" width="0" layer="19" extent="1-1"/>
+</signal>
+<signal name="ENC_A">
+<contactref element="XMC4800" pad="D2"/>
+<contactref element="R5" pad="2"/>
+<contactref element="R2" pad="1"/>
+<wire x1="1.27" y1="-15.24" x2="36.83" y2="27.94" width="0" layer="19" extent="1-1"/>
+<wire x1="13.97" y1="-34.29" x2="1.27" y2="-15.24" width="0" layer="19" extent="1-1"/>
+</signal>
+<signal name="ENC_B">
+<contactref element="XMC4800" pad="D3"/>
+<contactref element="R6" pad="2"/>
+<contactref element="R3" pad="1"/>
+<wire x1="1.27" y1="-21.59" x2="39.37" y2="27.94" width="0" layer="19" extent="1-1"/>
+<wire x1="13.97" y1="-40.64" x2="1.27" y2="-21.59" width="0" layer="19" extent="1-1"/>
+</signal>
 </signals>

Commit message: Board init design
Parts:
- added J1: (no value), uchile_robotics_eagle_lib:1X02_LOCK_LONGPADS
- moved HB_OUT 93.7 mm to (2.54, 12.7), turned to 270 degrees
- moved XMC4800 86.5 mm to (0.00, 20.3), turned to 0 degrees
- moved R6 78.3 mm to (34.3, 33.0), turned to 270 degrees
- moved R5 76.7 mm to (44.5, 33.0), turned to 270 degrees
- moved R4 68.7 mm to (39.4, 33.0), turned to 270 degrees
- moved HBRIDGE 52.8 mm to (61.0, 20.3), flipped to the bottom
- moved R2 49.5 mm to (44.5, 17.8), turned to 270 degrees
- moved R3 47.6 mm to (34.3, 17.8), turned to 270 degrees
- moved DB9 43.3 mm to (20.3, 6.35)
- moved R1 41.5 mm to (39.4, 17.8), turned to 270 degrees
- moved C1 28.4 mm to (16.5, 21.6), turned to 180 degrees
- moved CURRENT_SENSOR 24.2 mm to (19.1, 14.0), turned to 90 degrees
Connections:
- net +5V: now also J1.1
- net GND: now also J1.2
Routing:
- net N$3: track 0.00 -> 46.7 mm
- net GND: track 0.00 -> 27.7 mm
- net N$1: track 0.00 -> 23.4 mm, vias 0 -> 1
- net N$2: track 0.00 -> 12.3 mm, vias 0 -> 1
- net N$10: track 0.00 -> 11.1 mm
- net HOME: track 0.00 -> 2.54 mm
- net ENC_B: track 0.00 -> 2.54 mm
- net ENC_A: track 0.00 -> 2.54 mm
Other:
- board size 100 x 80 mm -> 61.9 x 82.5 mm

Commit message: Ruteo
Parts:
- moved J1 20.7 mm to (5.59, 25.7)
- moved C1 16.9 mm to (32.3, 15.5), turned to 270 degrees
- moved DB9 12.5 mm to (32.5, 9.14)
- moved R1 3.31 mm to (41.1, 20.6)
- moved R4 3.31 mm to (41.1, 35.8)
- moved HBRIDGE 3.31 mm to (62.7, 23.1)
- moved HB_OUT 3.31 mm to (4.32, 15.5)
- moved R2 3.31 mm to (46.2, 20.6)
- moved R3 3.31 mm to (36.1, 20.6)
- moved XMC4800 3.31 mm to (1.78, 23.1)
- moved CURRENT_SENSOR 3.31 mm to (20.8, 16.8)
- moved R5 3.31 mm to (46.2, 35.8)
- moved R6 3.31 mm to (36.1, 35.8)
Routing:
- net +5V: track 0.00 -> 147.3 mm
- net GND: track 27.7 -> 164.0 mm, vias 0 -> 2
- net INH2: track 0.00 -> 122.1 mm
- net INH1: track 0.00 -> 110.3 mm, vias 0 -> 1
- net IN1: track 0.00 -> 89.5 mm, vias 0 -> 1
- net ENC_A: track 2.54 -> 82.6 mm
- net IN2: track 0.00 -> 70.6 mm, vias 0 -> 1
- net HOME: track 2.54 -> 71.8 mm
- net ENC_B: track 2.54 -> 70.6 mm
- net !CS: track 0.00 -> 63.2 mm, vias 0 -> 1
- net +3V3: track 0.00 -> 60.2 mm, vias 0 -> 1
- net MISO: track 0.00 -> 57.3 mm, vias 0 -> 1
- net SCLK: track 0.00 -> 51.8 mm, vias 0 -> 1
- net N$11: track 0.00 -> 20.8 mm
- net N$1: track 23.4 -> 43.2 mm
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- added copper zone on layer 1, net GND
- added copper zone on layer 16, net GND
- added copper zone on layer 1, net N$5
Other:
- board size 61.9 x 82.5 mm -> 64.4 x 84.6 mm
- board text added: "+"
