Commit message: initial commit: ros-melodic rviz/gazebo scorbot model port. Added position/effort/trajectory controllers fro gazebo model. Added gripper.

File: ros/scorbot_description/robots/scorbot_pos.urdf.xacro (robot description, xacro)
@@ -20,11 +20,11 @@
   <xacro:gazebo_link link="left_finger" color="DarkGrey" />
   <!-- Transmissions -->
-  <xacro:joint_transmission joint="base"/>
-  <xacro:joint_transmission joint="shoulder"/>
-  <xacro:joint_transmission joint="elbow"/>
-  <xacro:joint_transmission joint="pitch"/>
+  <xacro:joint_pos_transmission joint="base"/>
+  <xacro:joint_pos_transmission joint="shoulder"/>
+  <xacro:joint_pos_transmission joint="elbow"/>
+  <xacro:joint_pos_transmission joint="pitch"/>
   <xacro:joint_pos_transmission joint="roll"/>
-  <xacro:joint_transmission joint="right_finger_tras"/>
-  <xacro:joint_transmission joint="left_finger_tras"/>
+  <xacro:joint_pos_transmission joint="right_finger_tras"/>
+  <xacro:joint_pos_transmission joint="left_finger_tras"/>
   <!-- Constants -->
   <xacro:property name="M_PI" value="3.14159265359" />
@@ -39,6 +39,6 @@
   <xacro:property name="pitch_upper_limit" value="${ 180.0/2*DEG2RAD}" />
   <xacro:property name="pitch_lower_limit" value="${-180.0/2*DEG2RAD}" />
-  <xacro:property name="roll_upper_limit" value="${  360.0/2*DEG2RAD}" />
-  <xacro:property name="roll_lower_limit" value="${- 360.0/2*DEG2RAD}" />
+  <xacro:property name="roll_upper_limit" value="${ 360.0/2*DEG2RAD}" />
+  <xacro:property name="roll_lower_limit" value="${-360.0/2*DEG2RAD}" />
   <xacro:property name="finger_upper_limit" value="${ 0.0165}" />
   <xacro:property name="finger_lower_limit" value="${-0.0165}" />

File: ros/scorbot_description/urdf/gazebo.urdf.xacro (robot description, xacro)
@@ -14,8 +14,8 @@
       <type>transmission_interface/SimpleTransmission</type>
       <joint name="${joint}">
-       <hardwareInterface>EffortJointInterface</hardwareInterface>
+       <hardwareInterface>hardware_interface/EffortJointInterface</hardwareInterface>
       </joint>
       <actuator name="${joint}_motor">
-        <hardwareInterface>EffortJointInterface</hardwareInterface>
+        <hardwareInterface>hardware_interface/EffortJointInterface</hardwareInterface>
         <mechanicalReduction>1</mechanicalReduction>
       </actuator>
@@ -27,8 +27,8 @@
       <type>transmission_interface/SimpleTransmission</type>
       <joint name="${joint}">
-       <hardwareInterface>PositionJointInterface</hardwareInterface>
+       <hardwareInterface>hardware_interface/PositionJointInterface</hardwareInterface>
       </joint>
       <actuator name="${joint}_motor">
-        <hardwareInterface>PositionJointInterface</hardwareInterface>
+        <hardwareInterface>hardware_interface/PositionJointInterface</hardwareInterface>
         <mechanicalReduction>1</mechanicalReduction>
       </actuator>
