Commit message: Add joint limits params

File: ros/scorbot_description/robots/scorbot.urdf.xacro (robot description, xacro)
@@ -23,4 +23,15 @@
   <xacro:joint_pos_transmission joint="pitch"/>
   <xacro:joint_pos_transmission joint="roll"/>
+  <!-- Joint limits in radians -->
+  <xacro:property name="base_upper_limit" value="1.0" />
+  <xacro:property name="base_lower_limit" value="-1.0" />
+  <xacro:property name="shoulder_upper_limit" value="1.0" />
+  <xacro:property name="shoulder_lower_limit" value="-1.0" />
+  <xacro:property name="elbow_upper_limit" value="1.0" />
+  <xacro:property name="elbow_lower_limit" value="-1.0" />
+  <xacro:property name="pitch_upper_limit" value="1.0" />
+  <xacro:property name="pitch_lower_limit" value="-1.0" />
+  <xacro:property name="roll_upper_limit" value="1.0" />
+  <xacro:property name="roll_lower_limit" value="-1.0" />
   <link
     name="base">
@@ -115,5 +126,5 @@
     <axis
       xyz="0 0 1" />
-    <limit effort="30" velocity="1.0" lower="-1.0" upper="1.0" />
+    <limit effort="30" velocity="1.0" lower="${base_lower_limit}" upper="${base_upper_limit}" />
   </joint>
   <link
@@ -169,5 +180,5 @@
     <axis
       xyz="0 1 0" />
-    <limit effort="30" velocity="1.0" lower="-1.0" upper="1.0" />
+    <limit effort="30" velocity="1.0" lower="${shoulder_lower_limit}" upper="${shoulder_upper_limit}" />
   </joint>
   <link
@@ -223,5 +234,5 @@
     <axis
       xyz="0 1 0" />
-    <limit effort="30" velocity="1.0" lower="-1.0" upper="1.0" />
+    <limit effort="30" velocity="1.0" lower="${elbow_lower_limit}" upper="${elbow_upper_limit}" />
   </joint>
   <link
@@ -277,5 +288,5 @@
     <axis
       xyz="0 1 0" />
-    <limit effort="30" velocity="1.0" lower="-1.0" upper="1.0" />
+    <limit effort="30" velocity="1.0" lower="${pitch_lower_limit}" upper="${pitch_upper_limit}" />
   </joint>
   <link name="tool" >
@@ -296,9 +307,8 @@
     <visual>
       <origin
-        xyz="0 0 0"
-        rpy="0 0 0" />
-      <geometry>
-        <mesh
-          filename="package://scorbot_description/meshes/flange.STL" />
+        xyz="0.05 0 0"
+        rpy="0 0 0" />
+      <geometry>
+        <box size="0.05 0.05 0.05"/>
       </geometry>
       <material
@@ -310,9 +320,8 @@
     <collision>
       <origin
-        xyz="0 0 0"
-        rpy="0 0 0" />
-      <geometry>
-        <mesh
-          filename="package://scorbot_description/meshes/flange.STL" />
+        xyz="0.05 0 0"
+        rpy="0 0 0" />
+      <geometry>
+        <box size="0.05 0.05 0.05"/>
       </geometry>
     </collision>
@@ -330,5 +339,5 @@
     <axis
       xyz="1 0 0" />
-    <limit effort="30" velocity="1.0" lower="-1.0" upper="1.0" />
+    <limit effort="30" velocity="1.0" lower="${roll_lower_limit}" upper="${roll_upper_limit}" />
   </joint>
 </robot>

Commit message: Add joint limits

File: ros/scorbot_description/robots/scorbot.urdf.xacro (robot description, xacro)
@@ -23,15 +23,18 @@
   <xacro:joint_pos_transmission joint="pitch"/>
   <xacro:joint_pos_transmission joint="roll"/>
+  <!-- Constants -->
+  <xacro:property name="M_PI" value="3.14159265359" />
+  <xacro:property name="DEG2RAD" value="${M_PI/180.0}" />
   <!-- Joint limits in radians -->
-  <xacro:property name="base_upper_limit" value="1.0" />
-  <xacro:property name="base_lower_limit" value="-1.0" />
-  <xacro:property name="shoulder_upper_limit" value="1.0" />
-  <xacro:property name="shoulder_lower_limit" value="-1.0" />
-  <xacro:property name="elbow_upper_limit" value="1.0" />
-  <xacro:property name="elbow_lower_limit" value="-1.0" />
-  <xacro:property name="pitch_upper_limit" value="1.0" />
-  <xacro:property name="pitch_lower_limit" value="-1.0" />
-  <xacro:property name="roll_upper_limit" value="1.0" />
-  <xacro:property name="roll_lower_limit" value="-1.0" />
+  <xacro:property name="base_upper_limit" value="${ 250.0/2*DEG2RAD}" />
+  <xacro:property name="base_lower_limit" value="${-250.0/2*DEG2RAD}" />
+  <xacro:property name="shoulder_upper_limit" value="${ 170.0/2*DEG2RAD}" />
+  <xacro:property name="shoulder_lower_limit" value="${-170.0/2*DEG2RAD}" />
+  <xacro:property name="elbow_upper_limit" value="${ 225.0/2*DEG2RAD}" />
+  <xacro:property name="elbow_lower_limit" value="${-225.0/2*DEG2RAD}" />
+  <xacro:property name="pitch_upper_limit" value="${ 180.0/2*DEG2RAD}" />
+  <xacro:property name="pitch_lower_limit" value="${-180.0/2*DEG2RAD}" />
+  <xacro:property name="roll_upper_limit" value="${ 360.0/2*DEG2RAD}" />
+  <xacro:property name="roll_lower_limit" value="${-360.0/2*DEG2RAD}" />
   <link
     name="base">

Commit message: Add dae for body and base

File: ros/scorbot_description/robots/scorbot.urdf.xacro (robot description, xacro)
@@ -56,8 +56,8 @@
       <origin
         xyz="0 0 0"
-        rpy="0 0 0" />
-      <geometry>
-        <mesh
-          filename="package://scorbot_description/meshes/base.STL" />
+        rpy="${M_PI/2.0} 0 0" />
+      <geometry>
+        <mesh
+          filename="package://scorbot_description/meshes/base.dae" />
       </geometry>
       <material
@@ -73,5 +73,5 @@
       <geometry>
         <mesh
-          filename="package://scorbot_description/meshes/base.STL" />
+          filename="package://scorbot_description/meshes/base.dae" />
       </geometry>
     </collision>
@@ -96,8 +96,8 @@
       <origin
         xyz="0 0 0"
-        rpy="0 0 0" />
-      <geometry>
-        <mesh
-          filename="package://scorbot_description/meshes/body.STL" />
+        rpy="${-M_PI/2.0} 0 0" />
+      <geometry>
+        <mesh
+          filename="package://scorbot_description/meshes/body.dae" />
       </geometry>
       <material

Commit message: Add dae frames

File: ros/scorbot_description/robots/scorbot.urdf.xacro (robot description, xacro)
@@ -150,8 +150,8 @@
       <origin
         xyz="0 0 0"
-        rpy="0 0 0" />
-      <geometry>
-        <mesh
-          filename="package://scorbot_description/meshes/upper_arm.STL" />
+        rpy="${-M_PI/2.0} 0 0" />
+      <geometry>
+        <mesh
+          filename="package://scorbot_description/meshes/upper_arm.dae" />
       </geometry>
       <material
@@ -204,8 +204,8 @@
       <origin
         xyz="0 0 0"
-        rpy="0 0 0" />
-      <geometry>
-        <mesh
-          filename="package://scorbot_description/meshes/forearm.STL" />
+        rpy="${M_PI/2.0} 0 0" />
+      <geometry>
+        <mesh
+          filename="package://scorbot_description/meshes/forearm.dae" />
       </geometry>
       <material
@@ -258,8 +258,8 @@
       <origin
         xyz="0 0 0"
-        rpy="0 0 0" />
-      <geometry>
-        <mesh
-          filename="package://scorbot_description/meshes/flange.STL" />
+        rpy="${-M_PI/2.0} 0 0" />
+      <geometry>
+        <mesh
+          filename="package://scorbot_description/meshes/flange.dae" />
       </geometry>
       <material

Commit message: Fix gripper TF

File: ros/scorbot_description/robots/scorbot.urdf.xacro (robot description, xacro)
@@ -70,5 +70,5 @@
       <origin
         xyz="0 0 0"
-        rpy="0 0 0" />
+        rpy="${M_PI/2.0} 0 0" />
       <geometry>
         <mesh
@@ -110,8 +110,8 @@
       <origin
         xyz="0 0 0"
-        rpy="0 0 0" />
-      <geometry>
-        <mesh
-          filename="package://scorbot_description/meshes/body.STL" />
+        rpy="${-M_PI/2.0} 0 0" />
+      <geometry>
+        <mesh
+          filename="package://scorbot_description/meshes/body.dae" />
       </geometry>
     </collision>
@@ -164,8 +164,8 @@
       <origin
         xyz="0 0 0"
-        rpy="0 0 0" />
-      <geometry>
-        <mesh
-          filename="package://scorbot_description/meshes/upper_arm.STL" />
+        rpy="${-M_PI/2.0} 0 0" />
+      <geometry>
+        <mesh
+          filename="package://scorbot_description/meshes/upper_arm.dae" />
       </geometry>
     </collision>
@@ -218,8 +218,8 @@
       <origin
         xyz="0 0 0"
-        rpy="0 0 0" />
-      <geometry>
-        <mesh
-          filename="package://scorbot_description/meshes/forearm.STL" />
+        rpy="${M_PI/2.0} 0 0" />
+      <geometry>
+        <mesh
+          filename="package://scorbot_description/meshes/forearm.dae" />
       </geometry>
     </collision>
@@ -272,8 +272,8 @@
       <origin
         xyz="0 0 0"
-        rpy="0 0 0" />
-      <geometry>
-        <mesh
-          filename="package://scorbot_description/meshes/flange.STL" />
+        rpy="${-M_PI/2.0} 0 0" />
+      <geometry>
+        <mesh
+          filename="package://scorbot_description/meshes/flange.dae" />
       </geometry>
     </collision>
@@ -283,5 +283,5 @@
     type="revolute">
     <origin
-      xyz="0.25 0.054 0"
+      xyz="0.25 0.058 0"
       rpy="0 0 0" />
     <parent
@@ -334,5 +334,5 @@
     type="revolute">
     <origin
-      xyz="0.054 -0.02 0"
+      xyz="0.054 -0.024 0"
       rpy="0 0 0" />
     <parent

Commit message: Add Gripper urdf based on dae files

File: ros/scorbot_description/robots/scorbot.urdf.xacro (robot description, xacro)
@@ -37,4 +37,7 @@
   <xacro:property name="roll_upper_limit" value="${ 360.0/2*DEG2RAD}" />
   <xacro:property name="roll_lower_limit" value="${-360.0/2*DEG2RAD}" />
+  <!-- Gripper joint limits -->
+  <xacro:property name="gripper_upper_limit" value="0.016" />
+  <xacro:property name="gripper_lower_limit" value="-0.018" />
   <link
     name="base">
@@ -293,41 +296,4 @@
     <limit effort="30" velocity="1.0" lower="${pitch_lower_limit}" upper="${pitch_upper_limit}" />
   </joint>
-  <link name="tool" >
-    <inertial>
-      <origin
-        xyz="0.0069957 -0.02 5.5511E-17"
-        rpy="0 0 0" />
-      <mass
-        value="0.24441" />
-      <inertia
-        ixx="0.00014819"
-        ixy="1.6491E-20"
-        ixz="-1.653E-19"
-        iyy="0.00028003"
-        iyz="5.3591E-21"
-        izz="0.00021086" />
-    </inertial>
-    <visual>
-      <origin
-        xyz="0.05 0 0"
-        rpy="0 0 0" />
-      <geometry>
-        <box size="0.05 0.05 0.05"/>
-      </geometry>
-      <material
-        name="">
-        <color
-          rgba="0.10196 0.10196 0.10196 1" />
-      </material>
-    </visual>
-    <collision>
-      <origin
-        xyz="0.05 0 0"
-        rpy="0 0 0" />
-      <geometry>
-        <box size="0.05 0.05 0.05"/>
-      </geometry>
-    </collision>
-  </link>
   <joint
     name="roll"
@@ -339,8 +305,157 @@
       link="flange" />
     <child
-      link="tool" />
+      link="gripper_base_link" />
     <axis
       xyz="1 0 0" />
     <limit effort="30" velocity="1.0" lower="${roll_lower_limit}" upper="${roll_upper_limit}" />
   </joint>
+  <!-- Gripper -->
+  <link
+    name="gripper_base_link">
+    <inertial>
+      <origin
+        xyz="0.0593648790750631 0 0"
+        rpy="0 0 0" />
+      <mass
+        value="1.59125921054032" />
+      <inertia
+        ixx="0.00147991252859225"
+        ixy="1.34230402513126E-19"
+        ixz="1.07467005492524E-19"
+        iyy="0.00232303179944379"
+        iyz="-4.07594317291221E-20"
+        izz="0.00291367454744379" />
+    </inertial>
+    <visual>
+      <origin
+        xyz="0 0 0"
+        rpy="${-M_PI/2.0} 0 0" />
+      <geometry>
+        <mesh
+          filename="package://scorbot_description/meshes/gripper_base.dae" />
+      </geometry>
+      <material
+        name="">
+        <color
+          rgba="0.898039215686275 0.917647058823529 0.929411764705882 1" />
+      </material>
+    </visual>
+    <collision>
+      <origin
+        xyz="0 0 0"
+        rpy="${-M_PI/2.0} 0 0" />
+      <geometry>
+        <mesh
+          filename="package://scorbot_description/meshes/gripper_base.dae" />
+      </geometry>
+    </collision>
+  </link>
+  <link
+    name="gripper_finger_left">
+    <inertial>
+      <origin
+        xyz="0.021935 0.017436 0.0038599"
+        rpy="0 0 0" />
+      <mass
+        value="0.1" />
+      <inertia
+        ixx="1.4677E-05"
+        ixy="-7.1238E-06"
+        ixz="3.6153E-06"
+        iyy="1.82E-05"
+        iyz="2.343E-06"
+        izz="2.4607E-05" />
+    </inertial>
+    <visual>
+      <origin
+        xyz="0 0 0"
+        rpy="${-M_PI/2.0} 0 0" />
+      <geometry>
+        <mesh
+          filename="package://scorbot_description/meshes/gripper_finger.dae" />
+      </geometry>
+      <material
+        name="">
+        <color
+          rgba="0.89804 0.91765 0.92941 1" />
+      </material>
+    </visual>
+    <collision>
+      <origin
+        xyz="0 0 0"
+        rpy="${-M_PI/2.0} 0 0" />
+      <geometry>
+        <mesh
+          filename="package://scorbot_description/meshes/gripper_finger.dae" />
+      </geometry>
+    </collision>
+  </link>
+  <joint
+    name="gripper_finger_left_joint"
+    type="prismatic">
+    <origin
+      xyz="0.118 0.0026 0.010"
+      rpy="0 0 0" />
+    <parent
+      link="gripper_base_link" />
+    <child
+      link="gripper_finger_left" />
+    <axis
+      xyz="0 1 0" />
+    <limit effort="30" velocity="1.0" lower="${gripper_lower_limit}" upper="${gripper_upper_limit}" />
+  </joint>
+  <link
+    name="gripper_finger_right">
+    <inertial>
+      <origin
+        xyz="0.021935 0.014436 -0.0061401"
+        rpy="0 0 0" />
+      <mass
+        value="0.1" />
+      <inertia
+        ixx="1.4677E-05"
+        ixy="-7.1238E-06"
+        ixz="3.6153E-06"
+        iyy="1.82E-05"
+        iyz="2.343E-06"
+        izz="2.4607E-05" />
+    </inertial>
+    <visual>
+      <origin
+        xyz="0 0 0"
+        rpy="${M_PI/2.0} 0 0" />
+      <geometry>
+        <mesh
+          filename="package://scorbot_description/meshes/gripper_finger.dae" />
+      </geometry>
+      <material
+        name="">
+        <color
+          rgba="0.89804 0.91765 0.92941 1" />
+      </material>
+    </visual>
+    <collision>
+      <origin
+        xyz="0 0 0"
+        rpy="${M_PI/2.0} 0 0" />
+      <geometry>
+        <mesh
+          filename="package://scorbot_description/meshes/gripper_finger.dae" />
+      </geometry>
+    </collision>
+  </link>
+  <joint
+    name="gripper_finger_right_joint"
+    type="prismatic">
+    <origin
+      xyz="0.118 -0.0026 -0.010"
+      rpy="0 0 0" />
+    <parent
+      link="gripper_base_link" />
+    <child
+      link="gripper_finger_right" />
+    <axis
+      xyz="0 -1 0" />
+    <limit effort="30" velocity="1.0" lower="${gripper_lower_limit}" upper="${gripper_upper_limit}" />
+  </joint>
 </robot>

Commit message: Add collition model based in basic shapes

File: ros/scorbot_description/robots/scorbot.urdf.xacro (robot description, xacro)
@@ -67,14 +67,17 @@
         name="">
         <color
-          rgba="0.49804 0.49804 0.49804 1" />
-      </material>
-    </visual>
-    <collision>
-      <origin
-        xyz="0 0 0"
-        rpy="${M_PI/2.0} 0 0" />
-      <geometry>
-        <mesh
-          filename="package://scorbot_description/meshes/base.dae" />
+          rgba="0.5 0.5 0.5 1" />
+      </material>
+    </visual>
+    <collision>
+      <origin rpy="0 0 0" xyz="0 0 0.0225"/>
+      <geometry>
+        <cylinder length="0.045" radius="0.16"/>
+      </geometry>
+    </collision>
+    <collision>
+      <origin rpy="0 0 0" xyz="0 0 0.085"/>
+      <geometry>
+        <cylinder length="0.170" radius="0.05"/>
       </geometry>
     </collision>
@@ -107,14 +110,11 @@
         name="">
         <color
-          rgba="0.49804 0.49804 0.49804 1" />
-      </material>
-    </visual>
-    <collision>
-      <origin
-        xyz="0 0 0"
-        rpy="${-M_PI/2.0} 0 0" />
-      <geometry>
-        <mesh
-          filename="package://scorbot_description/meshes/body.dae" />
+          rgba="0.5 0.5 0.5 1" />
+      </material>
+    </visual>
+    <collision>
+      <origin rpy="0 0 0" xyz="-0.08 0 0.125"/>
+      <geometry>
+        <box size="0.380 0.18 0.25"/>
       </geometry>
     </collision>
@@ -161,14 +161,11 @@
         name="">
         <color
-          rgba="0.49804 0.49804 0.49804 1" />
-      </material>
-    </visual>
-    <collision>
-      <origin
-        xyz="0 0 0"
-        rpy="${-M_PI/2.0} 0 0" />
-      <geometry>
-        <mesh
-          filename="package://scorbot_description/meshes/upper_arm.dae" />
+          rgba="0.5 0.5 0.5 1" />
+      </material>
+    </visual>
+    <collision>
+      <origin rpy="0 0 0" xyz="0.06 -0.06 0"/>
+      <geometry>
+        <box size="0.60 0.12 0.16"/>
       </geometry>
     </collision>
@@ -215,14 +212,11 @@
         name="">
         <color
-          rgba="0.49804 0.49804 0.49804 1" />
-      </material>
-    </visual>
-    <collision>
-      <origin
-        xyz="0 0 0"
-        rpy="${M_PI/2.0} 0 0" />
-      <geometry>
-        <mesh
-          filename="package://scorbot_description/meshes/forearm.dae" />
+          rgba="0.5 0.5 0.5 1" />
+      </material>
+    </visual>
+    <collision>
+      <origin rpy="0 0 0" xyz="0.05 0.035 0"/>
+      <geometry>
+        <box size="0.3 0.095 0.12"/>
       </geometry>
     </collision>
@@ -269,14 +263,11 @@
         name="">
         <color
-          rgba="0.10196 0.10196 0.10196 1" />
-      </material>
-    </visual>
-    <collision>
-      <origin
-        xyz="0 0 0"
-        rpy="${-M_PI/2.0} 0 0" />
-      <geometry>
-        <mesh
-          filename="package://scorbot_description/meshes/flange.dae" />
+          rgba="0.1 0.1 0.1 1" />
+      </material>
+    </visual>
+    <collision>
+      <origin rpy="${-M_PI/2.0} 0 0" xyz="0 -0.024 0"/>
+      <geometry>
+        <cylinder length="0.105" radius="0.05"/>
       </geometry>
     </collision>
@@ -338,14 +329,17 @@
         name="">
         <color
-          rgba="0.898039215686275 0.917647058823529 0.929411764705882 1" />
-      </material>
-    </visual>
-    <collision>
-      <origin
-        xyz="0 0 0"
-        rpy="${-M_PI/2.0} 0 0" />
-      <geometry>
-        <mesh
-          filename="package://scorbot_description/meshes/gripper_base.dae" />
+          rgba="0.1 0.1 0.1 1" />
+      </material>
+    </visual>
+    <collision>
+      <origin rpy="0 0 0" xyz="0.08 0.0 0.0"/>
+      <geometry>
+        <box size="0.078 0.110 0.055"/>
+      </geometry>
+    </collision>
+    <collision>
+      <origin rpy="0 ${-M_PI/2.0} 0" xyz="0.019 0 0"/>
+      <geometry>
+        <cylinder length="0.044" radius="0.05"/>
       </geometry>
     </collision>
@@ -378,5 +372,5 @@
         name="">
         <color
-          rgba="0.89804 0.91765 0.92941 1" />
+          rgba="0.9 0.9 0.9 1" />
       </material>
     </visual>
@@ -432,5 +426,5 @@
         name="">
         <color
-          rgba="0.89804 0.91765 0.92941 1" />
+          rgba="0.9 0.9 0.9 1" />
       </material>
     </visual>

Commit message: Fix description, remove old gripper

File: ros/scorbot_description/robots/scorbot.urdf.xacro (robot description, xacro)
@@ -14,15 +14,14 @@
   <xacro:gazebo_link link="forearm" color="White" />
   <xacro:gazebo_link link="flange" color="DarkGrey" />
-  <xacro:gazebo_link link="tool" color="DarkGrey" />
   <xacro:gazebo_link link="right_finger" color="DarkGrey" />
   <xacro:gazebo_link link="left_finger" color="DarkGrey" />
   <!-- Transmissions -->
-  <xacro:joint_transmission joint="base"/>
-  <xacro:joint_transmission joint="shoulder"/>
-  <xacro:joint_transmission joint="elbow"/>
-  <xacro:joint_transmission joint="pitch"/>
+  <xacro:joint_pos_transmission joint="base"/>
+  <xacro:joint_pos_transmission joint="shoulder"/>
+  <xacro:joint_pos_transmission joint="elbow"/>
+  <xacro:joint_pos_transmission joint="pitch"/>
   <xacro:joint_pos_transmission joint="roll"/>
-  <xacro:joint_transmission joint="right_finger_tras"/>
-  <xacro:joint_transmission joint="left_finger_tras"/>
+  <xacro:joint_transmission joint="gripper_finger_left_joint"/>
+  <xacro:joint_transmission joint="gripper_finger_right_joint"/>
   <!-- Constants -->
   <xacro:property name="M_PI" value="3.14159265359" />
@@ -42,8 +41,4 @@
   <xacro:property name="gripper_upper_limit" value="0.016" />
   <xacro:property name="gripper_lower_limit" value="-0.018" />
-  <xacro:property name="finger_upper_limit" value="${ 0.0165}" />
-  <xacro:property name="finger_lower_limit" value="${-0.0165}" />
-  <!-- * * * Define World Link to fix the arm's base to the world * * * -->
-  <link name="world"/>
   <link
     name="base">
@@ -459,113 +454,3 @@
     <limit effort="30" velocity="1.0" lower="${gripper_lower_limit}" upper="${gripper_upper_limit}" />
   </joint>
- <link name="right_finger" >
-    <inertial>
-      <origin
-        xyz="0.0219266 0.0154690 0.0037881"
-        rpy="0 0 0" />
-      <mass
-        value="0.019350" />
-      <inertia
-        ixx="545823883264E-17"
-        ixy="-263685619712E-17"
-        ixz="133104623616E-17"
-        iyy="675516317696E-17"
-        iyz="88172740608E-17"
-        izz="911899033600E-17" />
-    </inertial>
-	<visual>
-      <origin
-        xyz="0 0 0"
-        rpy="0 0 0" />
-      <geometry>
-        <mesh
-          filename="package://scorbot_description/meshes/right_finger.STL"/>
-      </geometry>
-      <material
-        name="">
-        <color
-          rgba="0.10196 0.10196 0.10196 1" />
-      </material>
-    </visual>
-    <collision>
-      <origin
-        xyz="0 0 0"
-        rpy="0 0 0" />
-      <geometry>
-        <mesh
-          filename="package://scorbot_description/meshes/right_finger.STL" />
-      </geometry>
-    </collision>
-  </link>
- <joint
-    name="right_finger_tras"
-    type="prismatic">
-    <origin
-      xyz="0.118 0 0"
-      rpy="0 0 0" />
-    <parent
-      link="tool" />
-    <child
-      link="right_finger" />
-    <axis
-      xyz="0 1 0" />
-    <limit effort="30" velocity="1.0" lower="${finger_lower_limit}" upper="${finger_upper_limit}" />
-  </joint>
-<link name="left_finger" >
-    <inertial>
-      <origin
-        xyz="0.0219266 -0.0154690 -0.0037881"
-        rpy="0 0 0" />
-      <mass
-        value="0.019350" />
-      <inertia
-        ixx="545823883264E-17"
-        ixy="263685619712E-17"
-        ixz="-133104623616E-17"
-        iyy="675516317696E-17"
-        iyz="88172740608E-17"
-        izz="911899033600E-17" />
-    </inertial>
-	<visual>
-      <origin
-        xyz="0 0 0"
-        rpy="0 0 0" />
-      <geometry>
-        <mesh
-          filename="package://scorbot_description/meshes/left_finger.STL" />
-      </geometry>
-      <material
-        name="">
-        <color
-          rgba="0.10196 0.10196 0.10196 1" />
-      </material>
-    </visual>
-    <collision>
-      <origin
-        xyz="0 0 0"
-        rpy="0 0 0" />
-      <geometry>
-        <mesh
-          filename="package://scorbot_description/meshes/left_finger.STL" />
-      </geometry>
-    </collision>
-  </link>
-<joint
-    name="left_finger_tras"
-    type="prismatic">
-    <origin
-      xyz="0.118 0 0"
-      rpy="0 0 0" />
-    <parent
-      link="tool" />
-    <child
-      link="left_finger" />
-    <axis
-      xyz="0 1 0" />
-    <limit effort="30" velocity="1.0" lower="${finger_lower_limit}" upper="${finger_upper_limit}" />
-  </joint>
-  <joint name="fixed" type="fixed">
-    <parent link="world"/>
-    <child link="base"/>
-  </joint>
 </robot>
