Commit message: Fix Scorbot gazebo ros_control for Indigo

File: ros/scorbot_description/robots/scorbot.urdf.xacro (robot description, xacro)
@@ -17,4 +17,5 @@
   <xacro:gazebo_link link="left_finger" color="DarkGrey" />
   <!-- Transmissions -->
+  <xacro:enable_ros_control prefix="scorbot/"/>
   <xacro:joint_pos_transmission joint="base"/>
   <xacro:joint_pos_transmission joint="shoulder"/>

File: ros/scorbot_description/urdf/gazebo.urdf.xacro (robot description, xacro)
@@ -2,5 +2,5 @@
 <robot xmlns:xacro="http://ros.org/wiki/xacro">
   <!-- ROS Control -->
-  <xacro:macro name="ros_control" params="prefix">
+  <xacro:macro name="enable_ros_control" params="prefix">
     <gazebo>
       <plugin filename="libgazebo_ros_control.so" name="ros_control">
@@ -14,8 +14,8 @@
       <type>transmission_interface/SimpleTransmission</type>
       <joint name="${joint}">
-       <hardwareInterface>hardware_interface/EffortJointInterface</hardwareInterface>
+       <hardwareInterface>EffortJointInterface</hardwareInterface>
       </joint>
       <actuator name="${joint}_motor">
-        <hardwareInterface>hardware_interface/EffortJointInterface</hardwareInterface>
+        <hardwareInterface>EffortJointInterface</hardwareInterface>
         <mechanicalReduction>1</mechanicalReduction>
       </actuator>
@@ -27,8 +27,8 @@
       <type>transmission_interface/SimpleTransmission</type>
       <joint name="${joint}">
-       <hardwareInterface>hardware_interface/PositionJointInterface</hardwareInterface>
+       <hardwareInterface>PositionJointInterface</hardwareInterface>
       </joint>
       <actuator name="${joint}_motor">
-        <hardwareInterface>hardware_interface/PositionJointInterface</hardwareInterface>
+        <hardwareInterface>PositionJointInterface</hardwareInterface>
         <mechanicalReduction>1</mechanicalReduction>
       </actuator>

Commit message: Fix gazebo sim deps, fix textures, add world to base fixed joint

File: ros/scorbot_description/robots/scorbot.urdf.xacro (robot description, xacro)
@@ -9,11 +9,11 @@
   <!-- Gazebo elements -->
   <!-- Gazebo Links material -->
-  <xacro:gazebo_link link="base" color="White" />
-  <xacro:gazebo_link link="body" color="White" />
-  <xacro:gazebo_link link="upper_arm" color="White" />
-  <xacro:gazebo_link link="forearm" color="White" />
-  <xacro:gazebo_link link="flange" color="DarkGrey" />
-  <xacro:gazebo_link link="right_finger" color="DarkGrey" />
-  <xacro:gazebo_link link="left_finger" color="DarkGrey" />
+  <xacro:gazebo_dae_link link="base" />
+  <xacro:gazebo_dae_link link="body" />
+  <xacro:gazebo_dae_link link="upper_arm" />
+  <xacro:gazebo_dae_link link="forearm" />
+  <xacro:gazebo_dae_link link="flange" />
+  <xacro:gazebo_dae_link link="right_finger" />
+  <xacro:gazebo_dae_link link="left_finger" />
   <!-- Transmissions -->
   <xacro:enable_ros_control prefix="scorbot/"/>
@@ -42,4 +42,10 @@
   <xacro:property name="gripper_upper_limit" value="0.016" />
   <xacro:property name="gripper_lower_limit" value="-0.018" />
+  <!-- Attach to the world frame -->
+  <link name="world"/>
+  <joint name="fixed" type="fixed">
+    <parent link="world"/>
+    <child link="base"/>
+  </joint>
   <link
     name="base">

File: ros/scorbot_description/urdf/gazebo.urdf.xacro (robot description, xacro)
@@ -36,5 +36,5 @@
   </xacro:macro>
   <!-- No gravity links -->
-  <xacro:macro name="gazebo_ng_link" params="link color">
+  <xacro:macro name="gazebo_no_gravity_link" params="link color">
     <gazebo reference="${link}">
       <material>Gazebo/${color}</material>
@@ -48,4 +48,11 @@
     <gazebo reference="${link}">
       <material>Gazebo/${color}</material>
+      <mu1>0.2</mu1>
+      <mu2>0.2</mu2>
+    </gazebo>
+  </xacro:macro>
+  <!-- Normal links DAE file -->
+  <xacro:macro name="gazebo_dae_link" params="link">
+    <gazebo reference="${link}">
       <mu1>0.2</mu1>
       <mu2>0.2</mu2>

Commit message: Test controller on scorbot

File: ros/scorbot_description/robots/scorbot.urdf.xacro (robot description, xacro)
@@ -42,10 +42,4 @@
   <xacro:property name="gripper_upper_limit" value="0.016" />
   <xacro:property name="gripper_lower_limit" value="-0.018" />
-  <!-- Attach to the world frame -->
-  <link name="world"/>
-  <joint name="fixed" type="fixed">
-    <parent link="world"/>
-    <child link="base"/>
-  </joint>
   <link
     name="base">

Commit message: Add tf prefix scorbot

File: ros/scorbot_description/robots/scorbot.urdf.xacro (robot description, xacro)
@@ -42,4 +42,11 @@
   <xacro:property name="gripper_upper_limit" value="0.016" />
   <xacro:property name="gripper_lower_limit" value="-0.018" />
+  <xacro:if value="$(arg fixed)">
+    <link name="world"/>
+    <joint name="fixed" type="fixed">
+      <parent link="world"/>
+      <child link="base"/>
+    </joint>
+  </xacro:if>
   <link
     name="base">
